Commit message: Added wheels to model

File: 24_02_2022/ws/src/puzzlebot_gazebo/urdf/puzzlebot.xacro (robot description, xacro)
@@ -58,13 +58,22 @@
   </joint>
 <!-- TASK 1a - create the shape needed for the wheel specified in  -->
- <!--RIGHT WHEEL
-	<link name="right_wheel">
-	</link> -->
+ <!-- RIGHT WHEEL  -->
+	<xacro:macro name="wheel" params="prefix roty">
+		<link name="${prefix}_wheel">
+			<visual>
+			<geometry>
+				<mesh filename="file://${mesh_wheel}"/>
+				<cylinder radius="${wheelRadius}" length="${wheelHeight}"/>
+			</geometry>
+			<origin xyz="0 0 0" rpy="${roty} 0 0"/>
+			</visual>
+		</link>
+	</xacro:macro>
+	<xacro:wheel prefix="right" roty="-1.57075" />
 <!-- TASK 1b -remember using Macros-->
-<!-- LEFT WHEEL
-	<link name="left_wheel">
-	</link> -->
+<!-- LEFT WHEEL  -->
+	<xacro:wheel prefix="left" roty="1.57075" />
 <!-- Remove comment to add joint -->
-<!-- JOINTS
+<!-- JOINTS    -->
   <joint name="base_to_right_w" type="continuous">
 	  <parent link="chassis" />
@@ -79,5 +88,4 @@
 	  <axis xyz="0 1 0" rpy="0 0 0" />
 	</joint>
--->
 <!-- TRANSMISSIONS (For a more complex model and it represents actuator attributes) -->
 </robot>

Commit message: Solve tasks 1 & 2

File: 24_02_2022/ws/src/puzzlebot_gazebo/urdf/puzzlebot.xacro (robot description, xacro)
@@ -5,8 +5,6 @@
 <xacro:include filename="$(find puzzlebot_gazebo)/urdf/parameters.xacro" />
 <xacro:include filename="$(find puzzlebot_gazebo)/urdf/macros.xacro" />
-<!--
 <xacro:include filename="$(find puzzlebot_gazebo)/urdf/puzzlebot.gazebo" />
 <xacro:include filename="$(find puzzlebot_gazebo)/urdf/materials.xacro" />
--->
 <!-- Dummy link needed to load the model properly-->
   <link name="base_link">
@@ -59,19 +57,29 @@
 <!-- TASK 1a - create the shape needed for the wheel specified in  -->
  <!-- RIGHT WHEEL  -->
-	<xacro:macro name="wheel" params="prefix roty">
+	<xacro:macro name="wheel" params="prefix">
 		<link name="${prefix}_wheel">
 			<visual>
-			<geometry>
-				<mesh filename="file://${mesh_wheel}"/>
-				<cylinder radius="${wheelRadius}" length="${wheelHeight}"/>
-			</geometry>
-			<origin xyz="0 0 0" rpy="${roty} 0 0"/>
+				<origin xyz="0 0 0" rpy="-${PI/2} 0 0" />
+				<geometry>
+					<mesh filename="file://${mesh_wheel}"/>
+				</geometry>
 			</visual>
+			<collision>
+				<origin xyz="0 0 0 " rpy="-${PI/2} 0 0"/>
+					<geometry>
+						<cylinder length="${wheelHeight}" radius="${wheelRadius}" />
+					</geometry>
+			</collision>
+			<inertial>
+				<mass value="${wheelMass}"/>
+				<origin xyz="0 0 0" rpy="${PI/2} 0 0"/>
+				<xacro:wheel_inertia r="${wheelRadius}" l="${wheelHeight}" m="${wheelMass}"/>
+			</inertial>
 		</link>
 	</xacro:macro>
-	<xacro:wheel prefix="right" roty="-1.57075" />
+	<xacro:wheel prefix="right"/>
 <!-- TASK 1b -remember using Macros-->
 <!-- LEFT WHEEL  -->
-	<xacro:wheel prefix="left" roty="1.57075" />
+	<xacro:wheel prefix="left"/>
 <!-- Remove comment to add joint -->
 <!-- JOINTS    -->
@@ -89,3 +97,23 @@
 	</joint>
 <!-- TRANSMISSIONS (For a more complex model and it represents actuator attributes) -->
+	<transmission name="right_wheel_trans">
+		<type>transmission_interface/SimpleTransmission</type>
+		<joint name="base_to_right_w">
+			<hardwareInterface>hardware_interface/VelocityJointInterface</hardwareInterface>
+		</joint>
+		<actuator name="right_wheel_motor">
+		<mechanicalReduction>34</mechanicalReduction>
+		<hardwareInterface>hardware_interface/VelocityJointInterface</hardwareInterface>
+		</actuator>
+	</transmission>
+	<transmission name="left_wheel_trans">
+		<type>transmission_interface/SimpleTransmission</type>
+		<joint name="base_to_left_w">
+			<hardwareInterface>hardware_interface/VelocityJointInterface</hardwareInterface>
+		</joint>
+		<actuator name="left_wheel_motor">
+		<mechanicalReduction>34</mechanicalReduction>
+		<hardwareInterface>hardware_interface/VelocityJointInterface</hardwareInterface>
+		</actuator>
+	</transmission>
 </robot>
